File: 1515/APA102/APA102-1515-6_8x8_matrix.kicad_pcb (KiCad board)
At the start: 4 copper layers, 24 x 24 mm, 85 parts, among them J1 INPUT_CONN, J2 OUTPUT_CONN, J3 INPUT_CONN, J4 OUTPUT_CONN, J5 POWER_CONN

Commit message: .
Parts:
- J5: footprint _kicad_selfmadeStandartFootprint:Conn_Molex_2026560021(Pico-EZmate_Slim) -> _conn:Conn_Molex_2026560021(Pico-EZmate_Slim)
